File: board/cheapbmc.kicad_pcb (KiCad board)
At the start: 2 copper layers, 57.2 x 46.4 mm, 22 parts, among them J1 Conn_01x02_Male, J2 atxpanel, J3 atxpanel, J4 Conn_01x03_Male, K1 SILxx-1Axx-71x, K2 SILxx-1Axx-71x, Q1 BC547, Q2 BC547, SW1 SW_Push, U1 NodeMCU1.0(ESP-12E)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

Commit message: Move connector away from mounting hole
Parts:
- moved J1 1.27 mm to (113.0, 44.5)
Routing:
- net Net-(J1-Pad1): track 48.9 -> 50.2 mm
